Commit message: Add static mission planner and alter naming convention

File: usv_simulator/config/models/viknes.urdf (robot description, URDF)
Before this commit: robot usv, 1 links, 0 joints
Links:
- removed link usv
- added link Viknes830; visual mesh filename=package://usv_simulator/meshes/viknes.STL scale=0.001 0.001 0.001
