Commit message: Add obstacle ship and mock tracking

File: usv_simulator/config/models/ship1.urdf (robot description, URDF)
Before this commit: robot ship1, 1 links, 0 joints
Links:
- removed link obstacles/ship1
- added link ship1; visual mesh filename=package://asv_simulator/meshes/Revolt.STL scale=0.0001 0.0001 0.0001

Commit message: Working head-on scenario

File: usv_simulator/config/models/ship1.urdf (robot description, URDF)
Before this commit: robot ship1, 1 links, 0 joints
Links:
- link ship1: geometry visual mesh filename=package://usv_simulator/meshes/viknes.STL scale=0.001 0.001 0.001
